Commit message: fix: weight, curve, reward

File: assets/f1tenth/f1tenth.urdf (robot description, URDF)
Before this commit: robot f1tenth, 7 links, 6 joints
Links:
- link base_link: mass 3.441 -> 3.741

Commit message: fix: weight, noise

File: assets/f1tenth/f1tenth.urdf (robot description, URDF)
Before this commit: robot f1tenth, 7 links, 6 joints
Links:
- link base_link: mass 3.741 -> 4.032

Commit message: fix: weight

File: assets/f1tenth/f1tenth.urdf (robot description, URDF)
Before this commit: robot f1tenth, 7 links, 6 joints
Links:
- link base_link: mass 4.032 -> 4.487
